File: hardware/PCB/esp32-ups-snmp/esp32-ups-snmp.kicad_sch (KiCad schematic)
At the start: 2 parts, among them J1 USB_A

Commit message: WIP on HTTP OTA
Parts:
- J1: footprint Connector_USB:USB_A_Kycon_KUSBX-AS1N-B_Horizontal -> Connector_USB:USB_A_Wuerth_614004134726_Horizontal
Changed lines of the file:
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@@
 			)
 		)
-		(property "Footprint" "Connector_USB:USB_A_Kycon_KUSBX-AS1N-B_Horizontal"
+		(property "Footprint" "Connector_USB:USB_A_Wuerth_614004134726_Horizontal"
 			(at 179.07 54.61 0)
 			(effects
